File: LT3652EvalBoard.kicad_pcb (KiCad board)
At the start: 2 copper layers, 49.8 x 49.8 mm, 46 parts, among them U1 LT3652

Commit message: Rev 0.10
Parts:
- removed Dvin2: ZLLS500, ms_diodes:DIODES_INC_ZLLS500
- removed JPnl1: JUMPER3, Pin_Headers:Pin_Header_Straight_1x03
- removed Pslr3: JST PH, w_conn_jst-ph:b2b-ph-kl
- added JP4: Jumper_NO_Small, Resistors_SMD:R_0805_HandSoldering, F.Cu at (133.1, 68.8)
- added JP5: Jumper_NC_Small, Resistors_SMD:R_0805_HandSoldering, F.Cu at (133.1, 72.5)
- added Wbst1: TEST_1P, Measurement_Points:Measurement_Point_Round-SMD-Pad_Small, F.Cu at (142.5, 85.5)
- added Wsw2: TEST_1P, Measurement_Points:Measurement_Point_Round-SMD-Pad_Small, F.Cu at (135.3, 89.2)
- moved Pslr2 16.4 mm to (140.8, 68.8)
- moved Dvin1 7.91 mm to (122.9, 72.8)
- moved Pslr1 7.70 mm to (125.0, 68.8)
- moved Dflybk1 1.30 mm to (133.2, 86.8)
Routing:
- net GND: track 12.4 -> 22.7 mm
- net Net-(JP4-Pad1): track 17.7 -> 9.45 mm
- net Net-(JPnl1-Pad3): track 7.87 -> 0.00 mm
- net /VIN: track 116.4 -> 111.9 mm
- net Net-(Dvin1-Pad3): track 4.22 -> 3.16 mm
- net Net-(JP4-Pad2): track 6.25 -> 5.35 mm
- net /SW: track 26.4 -> 27.1 mm
Other:
- board text added: "LT3652 Eval Board Rev 0.10 27-02-2017"
- board text removed: "GND"
- board text removed: "LT3652 Eval Board Rev 0.9 10-04-2016"
- board text removed: "SER"
